Commit message: urdf now defined

File: src/CRAP_sim_def/urdf/CRAP.xacro (robot description, xacro)
@@ -1,4 +1,4 @@
 <?xml version="1.0"?>
-<robot xmlns:xacro="http://www.ros.org/wiki/xacro" name="mecanum_robot">
+<robot xmlns:xacro="http://www.ros.org/wiki/xacro" name="CRAP">
   <!-- Define the base link of the robot -->
   <link name="base_link">
@@ -11,5 +11,5 @@
       <origin xyz="0 0 0" rpy="0 0 0"/>
       <geometry>
-        <box size="0.5 0.5 0.1"/>
+        <box size="0.5 0.5 0.05"/>
       </geometry>
       <material name="red">
@@ -18,19 +18,31 @@
     </visual>
   </link>
-  <!-- Define the four mecanum wheels -->
-  <xacro:include filename="$(find CRAP_sim_def)/urdf/wheel.xacro"/>
-  <wheel name="front_left_wheel" parent="base_link" x="0.25" y="0.25" />
-  <wheel name="front_right_wheel" parent="base_link" x="0.25" y="-0.25" />
-  <wheel name="rear_left_wheel" parent="base_link" x="-0.25" y="0.25" />
-  <wheel name="rear_right_wheel" parent="base_link" x="-0.25" y="-0.25" />
+  <!-- Define the four  wheels -->
+  <xacro:include filename="wheel.xacro"/>
+  <xacro:wheel name="front_left_wheel" parent="base_link" x="0.25" y="0.25" />
+  <xacro:wheel name="front_right_wheel" parent="base_link" x="0.25" y="-0.25" />
+  <xacro:wheel name="rear_left_wheel" parent="base_link" x="-0.25" y="0.25" />
+  <xacro:wheel name="rear_right_wheel" parent="base_link" x="-0.25" y="-0.25" />
   <!-- Define the LIDAR sensor -->
-  <xacro:include filename="$(find CRAP_sim_def)/urdf/lidar.xacro"/>
-  <lidar name="hokuyo" parent="base_link" x="0" y="0" z="0.2" />
-  <!-- Define the stereo camera -->
-  <!-- <xacro:include filename="$(find sCRAP_sim_def)/urdf/stereo_camera.xacro"/>
-  <stereo_camera name="stereo_camera_sensor" parent="base_link" x="0" y="0" z="0.1" /> -->
+  <xacro:include filename="lidar_gazebo.xacro"/>
+  <xacro:rplidar prefix="lidar" parent="base_link" x="0" y="0" z="0.05"/>
   <!-- Define the rgbd camera -->
-  <!-- <xacro:include filename="$(find sCRAP_sim_def)/urdf/stereo_camera.xacro"/>
-  <stereo_camera name="stereo_camera_sensor" parent="base_link" x="0" y="0" z="0.1" /> -->
-  <xacro:include filename="$(find CRAP_sim_def)/urdf/CRAP.gazebo" />
+  <xacro:include filename="kinect_gazebo.xacro"/>
+  <xacro:kinect_camera prefix="kinect" parent="base_link" x="0.27" y="0" z="0"/>
+  <gazebo>
+    <plugin name="skid_steer_drive_controller" filename="libgazebo_ros_skid_steer_drive.so">
+      <updateRate>100.0</updateRate>
+      <robotNamespace>/</robotNamespace>
+      <leftFrontJoint>front_left_wheel_joint</leftFrontJoint>
+      <rightFrontJoint>front_right_wheel_joint</rightFrontJoint>
+      <leftRearJoint>back_left_wheel_joint</leftRearJoint>
+      <rightRearJoint>back_right_wheel_joint</rightRearJoint>
+      <wheelSeparation>0.5</wheelSeparation>
+      <wheelDiameter>0.2</wheelDiameter>
+      <robotBaseFrame>base_link</robotBaseFrame>
+      <torque>10</torque>
+      <topicName>cmd_vel</topicName>
+      <broadcastTF>false</broadcastTF>
+    </plugin>
+  </gazebo>
 </robot>

File: src/CRAP_sim_def/urdf/wheel.xacro (robot description, xacro)
@@ -1,38 +1,41 @@
 <?xml version="1.0"?>
-<robot xmlns:xacro="http://www.ros.org/wiki/xacro" name="wheel">
-  <!-- Define the wheel link -->
-  <link name="${name}_link">
-    <inertial>
-      <mass value="1.0"/>
-      <origin xyz="0 0 0" rpy="0 1.5707 1.5707"/>
-      <inertia ixx="0.005" ixy="0" ixz="0" iyy="0.005" iyz="0" izz="0.005"/>
-    </inertial>
-    <visual>
-      <origin xyz="0 0 0" rpy="0 0 0"/>
-      <geometry>
-        <cylinder radius="${robot_wheel_radius}" length="${robot_wheel_radius}"/>
-      </geometry>
-      <material name="black">
-        <color rgba="0 0 0 1"/>
-      </material>
-    </visual>
-  </link>
-  <!-- Define the wheel joint -->
-  <joint name="${name}_joint" type="continuous">
-    <origin xyz="${x} ${y} 0" rpy="0 0 0"/>
-    <parent link="${parent}"/>
-    <child link="${name}_link"/>
-    <axis xyz="0 1 0"/>
-    <limit effort="10000" velocity="1000" />
-	  <dynamics damping="1.0" friction="1.0" />
-  </joint>
-	<gazebo reference="${name}_link">
-		<material>Gazebo/Green</material>
-		<kp>1000000.0</kp> <!-- kp and kd for rubber -->
-		<kd>100.0</kd>
-		<mu1>1.0</mu1>
-		<mu2>1.0</mu2>
-		<maxVel>1.0</maxVel>
-		<minDepth>0.00</minDepth>
-	</gazebo>
+<robot xmlns:xacro="http://www.ros.org/wiki/xacro" name="wheel_macro">
+  <xacro:property name="M_PI" value="3.141592653589793"/>
+  <xacro:macro name="wheel" params="name parent x y">
+    <!-- Define the wheel link -->
+    <link name="${name}_link">
+      <inertial>
+        <mass value="1.0"/>
+        <origin xyz="0 0 0" rpy="0 ${M_PI/2} ${M_PI/2}"/>
+        <inertia ixx="0.005" ixy="0" ixz="0" iyy="0.005" iyz="0" izz="0.005"/>
+      </inertial>
+      <visual>
+        <origin xyz="0 0 0" rpy="0 ${M_PI/2} ${M_PI/2}"/>
+        <geometry>
+          <cylinder radius="0.05" length="0.02"/>
+        </geometry>
+        <material name="black">
+          <color rgba="0 0 0 1"/>
+        </material>
+      </visual>
+    </link>
+    <!-- Define the wheel joint -->
+    <joint name="${name}_joint" type="continuous">
+      <origin xyz="${x} ${y} 0" rpy="0 0 0"/>
+      <parent link="${parent}"/>
+      <child link="${name}_link"/>
+      <axis xyz="0 1 0"/>
+      <limit effort="10000" velocity="1000" />
+      <dynamics damping="1.0" friction="1.0" />
+    </joint>
+    <gazebo reference="${name}_link">
+      <material>Gazebo/Green</material>
+      <kp>1000000.0</kp> <!-- kp and kd for rubber -->
+      <kd>100.0</kd>
+      <mu1>1.0</mu1>
+      <mu2>1.0</mu2>
+      <maxVel>1.0</maxVel>
+      <minDepth>0.00</minDepth>
+    </gazebo>
+  </xacro:macro>
 </robot>

Commit message: got gazebo running at last

File: src/CRAP_sim_def/urdf/CRAP.xacro (robot description, xacro)
@@ -2,4 +2,19 @@
 <robot xmlns:xacro="http://www.ros.org/wiki/xacro" name="CRAP">
   <!-- Define the base link of the robot -->
+    <link name="base_footprint">
+      <visual>
+          <origin xyz="0 0 0" rpy="0 0 0" />
+          <geometry>
+              <box size="0.001 0.001 0.001" />
+          </geometry>
+      </visual>
+  </link>
+  <gazebo reference="base_footprint">
+      <turnGravityOff>false</turnGravityOff>
+  </gazebo>
+  <joint name="base_footprint_joint" type="fixed">
+      <parent link="base_footprint"/>
+      <child link="base_link" />
+  </joint>
   <link name="base_link">
     <inertial>
@@ -17,4 +32,9 @@
       </material>
     </visual>
+    <collision>
+      <geometry>
+          <box size="0.5 0.5 0.05"/>
+      </geometry>
+    </collision>
   </link>
   <!-- Define the four  wheels -->
@@ -31,5 +51,31 @@
   <xacro:kinect_camera prefix="kinect" parent="base_link" x="0.27" y="0" z="0"/>
   <gazebo>
-    <plugin name="skid_steer_drive_controller" filename="libgazebo_ros_skid_steer_drive.so">
+      <plugin name='skid_steer_drive' filename='libgazebo_ros_diff_drive.so'>
+      <!-- Update rate -->
+      <update_rate>100</update_rate>
+      <!-- Number of wheel pairs -->
+      <num_wheel_pairs>2</num_wheel_pairs>
+      <!-- wheels0 -->
+      <left_joint>front_left_wheel_joint</left_joint>
+      <right_joint>front_right_wheel_joint</right_joint>
+      <!-- wheels1-->
+      <left_joint>rear_left_wheel_joint</left_joint>
+      <right_joint>rear_right_wheel_joint</right_joint>
+      <!-- kinematics -->
+      <wheel_separation>0.5</wheel_separation>
+      <wheel_separation>0.5</wheel_separation>
+      <wheel_diameter>0.1</wheel_diameter>
+      <wheel_diameter>0.1</wheel_diameter>
+      <!-- limits -->
+      <max_wheel_torque>20</max_wheel_torque>
+      <max_wheel_acceleration>1.0</max_wheel_acceleration>
+      <!-- output -->
+      <publish_odom>true</publish_odom>
+      <publish_odom_tf>true</publish_odom_tf>
+      <publish_wheel_tf>true</publish_wheel_tf>
+      <odometry_frame>odom</odometry_frame>
+      <robot_base_frame>base_link</robot_base_frame>
+      </plugin>
+    <!-- <plugin name="skid_steer_drive_controller" filename="libgazebo_ros_skid_steer_drive.so">
       <updateRate>100.0</updateRate>
       <robotNamespace>/</robotNamespace>
@@ -43,6 +89,15 @@
       <torque>10</torque>
       <topicName>cmd_vel</topicName>
-      <broadcastTF>false</broadcastTF>
-    </plugin>
+      <odometryTopic>odom</odometryTopic>
+      <odometryFrame>odom</odometryFrame>
+      <commandTopic>cmd_vel</commandTopic>
+      <topic_name_twist>cmd_vel</topic_name_twist>
+      <topic_name_odometry>odom</topic_name_odometry>
+      <topic_name_joint>joint</topic_name_joint>
+      <broadcastTF>true</broadcastTF>
+      <covariance_x>0.0001</covariance_x>
+      <covariance_y>0.0001</covariance_y>
+      <covariance_yaw>0.01</covariance_yaw>
+    </plugin> -->
   </gazebo>
 </robot>

File: src/CRAP_sim_def/urdf/lidar_gazebo.xacro (robot description, xacro)
@@ -16,5 +16,7 @@
                     <cylinder length="0.05" radius="0.05"/>
                 </geometry>
-                <material name="green"/>
+                <material name="green">
+                    <color rgba="0 1 0 1"/>
+                </material>
             </visual>
             <collision>

File: src/CRAP_sim_def/urdf/wheel.xacro (robot description, xacro)
@@ -2,4 +2,6 @@
 <robot xmlns:xacro="http://www.ros.org/wiki/xacro" name="wheel_macro">
   <xacro:property name="M_PI" value="3.141592653589793"/>
+  <xacro:property name="radius" value="0.05"/>
+  <xacro:property name="thickness" value="0.02"/>
   <xacro:macro name="wheel" params="name parent x y">
     <!-- Define the wheel link -->
@@ -13,5 +15,5 @@
         <origin xyz="0 0 0" rpy="0 ${M_PI/2} ${M_PI/2}"/>
         <geometry>
-          <cylinder radius="0.05" length="0.02"/>
+          <cylinder radius="${radius}" length="${thickness}"/>
         </geometry>
         <material name="black">
@@ -19,4 +21,10 @@
         </material>
       </visual>
+      <collision>
+        <origin xyz="0.0 0.0 0.0" rpy="0 ${M_PI/2} ${M_PI/2}" />
+          <geometry>
+              <cylinder length="${thickness}" radius="${radius}"/>
+          </geometry>
+      </collision>
     </link>
     <!-- Define the wheel joint -->
@@ -30,5 +38,5 @@
     </joint>
     <gazebo reference="${name}_link">
-      <material>Gazebo/Green</material>
+      <material>Gazebo/Blue</material>
       <kp>1000000.0</kp> <!-- kp and kd for rubber -->
       <kd>100.0</kd>
@@ -38,4 +46,14 @@
       <minDepth>0.00</minDepth>
     </gazebo>
+    <transmission name="${name}_wheel_joint_trans">
+        <type>transmission_interface/SimpleTransmission</type>
+        <joint name="${name}_joint" >
+            <hardwareInterface>hardware_interface/VelocityJointInterface</hardwareInterface>
+        </joint>
+        <actuator name="${name}_joint_motor">
+            <hardwareInterface>hardware_interface/VelocityJointInterface</hardwareInterface>
+            <mechanicalReduction>1</mechanicalReduction>
+        </actuator>
+    </transmission>
   </xacro:macro>
 </robot>
